Commit message: reconfigured simulated sensors to match real sensors

File: blue_description/description/bluerov2/sensors.xacro (robot description, xacro)
@@ -5,5 +5,6 @@
     <xacro:include filename="$(find blue_description)/description/vn100/urdf.xacro" />
     <xacro:imu_urdf prefix="$(arg prefix)" parent="$(arg prefix)base_link">
-      <origin rpy="0 0 0" xyz="0.0 0.0 0.1" />
+      <!-- Should output body-fixed measurements(NED)-->
+      <origin rpy="3.1415 0 0" xyz="0.0 0.0 0.1" />
     </xacro:imu_urdf>
     <!-- Import DVL sensor -->
@@ -15,5 +16,6 @@
     <xacro:if value="$(arg use_sim)">
       <xacro:include filename="$(find blue_description)/description/vn100/gazebo.xacro" />
-      <xacro:imu_gazebo reference="$(arg prefix)imu_link" topic="/vn100/gz_data" frame_id="imu_link" />
+      <xacro:imu_gazebo reference="$(arg prefix)imu_link" topic="/vectornav/Imu_body"
+        frame_id="vectornav" />
       <xacro:include filename="$(find blue_description)/description/dvl/gazebo.xacro" />
       <xacro:dvl_gazebo reference="$(arg prefix)dvl_link" topic="/dvl/data_test" />

File: blue_description/description/vn100/gazebo.xacro (robot description, xacro)
@@ -1,5 +1,5 @@
 <?xml version="1.0"?>
 <robot xmlns:xacro="http://ros.org/wiki/xacro">
-  <xacro:macro name="imu_gazebo" params="reference topic:=vn100_data frame_id:=imu_link">
+  <xacro:macro name="imu_gazebo" params="reference topic:=vn100_data frame_id:=vectornav">
     <gazebo reference="${reference}">
       <sensor name="vn100" type="imu">

Commit message: Removed use of EK3 in Ros2 EKF

File: blue_description/description/bluerov2/sensors.xacro (robot description, xacro)
@@ -11,5 +11,5 @@
     <xacro:include filename="$(find blue_description)/description/dvl/urdf.xacro" />
     <xacro:dvl_urdf prefix="$(arg prefix)" parent="$(arg prefix)base_link">
-      <origin rpy="3.1416 0 0" xyz="0.0 0.0 -0.2" />
+      <origin rpy="3.1416 0 0" xyz="0.0 0.0 -0.12" />
     </xacro:dvl_urdf>
     <!-- Add Gazebo sensor plugins if in simulation -->

File: blue_description/description/dvl/urdf.xacro (robot description, xacro)
@@ -4,5 +4,5 @@
     <link name="${prefix}dvl_link">
       <inertial>
-        <mass value="0.170" />
+        <mass value="0.0170" />
         <inertia
           ixx="0.00005514"

File: blue_description/description/vn100/gazebo.xacro (robot description, xacro)
@@ -40,9 +40,7 @@
               <noise type="gaussian">
                 <mean>0.0</mean>
-                <!-- <stddev>0.013734</stddev> -->
-                <stddev>0.0</stddev>
+                <stddev>0.013734</stddev>
                 <bias_mean>0.0</bias_mean>
-                <!-- <bias_stddev>0.0003924</bias_stddev> -->
-                <bias_stddev>0.00</bias_stddev>
+                <bias_stddev>0.0003924</bias_stddev>
               </noise>
             </x>
@@ -50,9 +48,7 @@
               <noise type="gaussian">
                 <mean>0.0</mean>
-                <!-- <stddev>0.013734</stddev> -->
-                <stddev>0.0</stddev>
+                <stddev>0.013734</stddev>
                 <bias_mean>0.0</bias_mean>
-                <!-- <bias_stddev>0.0003924</bias_stddev> -->
-                <bias_stddev>0.00</bias_stddev>
+                <bias_stddev>0.0003924</bias_stddev>
               </noise>
             </y>
@@ -60,9 +56,7 @@
               <noise type="gaussian">
                 <mean>0.0</mean>
-                <!-- <stddev>0.013734</stddev> -->
-                <stddev>0.0</stddev>
+                <stddev>0.013734</stddev>
                 <bias_mean>0.0</bias_mean>
-                <!-- <bias_stddev>0.0003924</bias_stddev> -->
-                <bias_stddev>0.00</bias_stddev>
+                <bias_stddev>0.0003924</bias_stddev>
               </noise>
             </z>

File: blue_description/description/vn100/urdf.xacro (robot description, xacro)
@@ -4,5 +4,5 @@
     <link name="${prefix}imu_link">
       <inertial>
-        <mass value="0.015" />
+        <mass value="0.00015" />
         <inertia
           ixx="0.0000017"
